Commit message: sensor incomplete

File: model_description/urdf/mkz_13_structure.urdf.xacro (robot description, xacro)
@@ -2,4 +2,7 @@
 <!-- created with Phobos 0.7 -->
   <robot name="dbw_mkz" xmlns:xacro="http://www.ros.org/wiki/xacro">
+    <xacro:include filename="$(find model_description)/urdf/materials.xacro" />
+    <xacro:include filename="$(find model_description)/urdf/model.gazebo" />
+    <xacro:include filename="$(find model_description)/urdf/model.trans" />
     <link name="base_footprint">
     </link>
@@ -7,6 +10,6 @@
       <inertial>
         <origin xyz="1.4225 0 0.25" rpy="0 0 0"/>
-        <mass value="1500.0"/>
-        <inertia ixx="1000.0" ixy="0" ixz="0" iyy="1000.0" iyz="0" izz="1000.0"/>
+        <mass value="0.2"/>
+        <inertia ixx="0.1" ixy="0.0" ixz="0.0" iyy="0.1" iyz="0.0" izz="0.1"/>
       </inertial>
       <visual name="chassis">
@@ -118,4 +121,64 @@
       </collision>
     </link>
+    <!-- Camera -->
+    <link name="camera_link">
+      <collision>
+        <origin xyz="0 0 0" rpy="0 0 0"/>
+        <geometry>
+          <box size="0.05 0.05 0.05"/>
+        </geometry>
+      </collision>
+      <visual>
+        <origin xyz="0 0 0" rpy="0 0 0"/>
+        <geometry>
+          <box size="0.05 0.05 0.05"/>
+        </geometry>
+      </visual>
+      <inertial>
+        <origin xyz="0 0 0" rpy="0 0 0"/>
+        <mass value="0.1"/>
+        <inertia ixx="1" ixy="1" ixz="1.0" iyy="1.0" iyz="1.0" izz="1.0"/>
+      </inertial>
+    </link>
+    <!-- gps -->
+    <link name="gps_link">
+      <collision>
+        <origin xyz="0 0 0" rpy="0 0 0"/>
+        <geometry>
+          <box size="0.05 0.05 0.05"/>
+        </geometry>
+      </collision>
+      <visual>
+        <origin xyz="0 0 0" rpy="0 0 0"/>
+        <geometry>
+          <box size="0.05 0.05 0.05"/>
+        </geometry>
+      </visual>
+      <inertial>
+        <origin xyz="0 0 0" rpy="0 0 0"/>
+        <mass value="0.1"/>
+        <inertia ixx="1" ixy="1" ixz="1.0" iyy="1.0" iyz="1.0" izz="1.0"/>
+      </inertial>
+    </link>
+  <!-- lidar -->
+    <link name="sensor_laser">
+    <inertial>
+        <origin xyz="0 0 0" rpy="0 0 0"/>
+        <mass value="0.1"/>
+        <inertia ixx="1" ixy="1" ixz="1.0" iyy="1.0" iyz="1.0" izz="1.0"/>
+    </inertial>
+    <visual>
+        <origin xyz="0 0 0" rpy="0 0 0" />
+        <geometry>
+        <cylinder radius="0.025" length="0.05"/>
+        </geometry>
+    </visual>
+    <collision>
+        <origin xyz="0 0 0" rpy="0 0 0"/>
+        <geometry>
+        <cylinder radius="0.05" length="0.1"/>
+        </geometry>
+    </collision>
+  </link>
     <joint name="base_link_joint" type="fixed">
       <origin xyz="0 0 0.33" rpy="0 0 0"/>
@@ -142,5 +205,5 @@
       <child link="wheel_fl"/>
       <axis xyz="0 0 1.0"/>
-      <limit effort="0" velocity="22.0"/>
+      <limit effort="10" velocity="22.0"/>
     </joint>
     <joint name="wheel_fr_joint" type="continuous">
@@ -149,5 +212,5 @@
       <child link="wheel_fr"/>
       <axis xyz="0 0 1.0"/>
-      <limit effort="0" velocity="22.0"/>
+      <limit effort="10" velocity="22.0"/>
     </joint>
     <joint name="wheel_rl_joint" type="continuous">
@@ -156,5 +219,5 @@
       <child link="wheel_rl"/>
       <axis xyz="0 0 1.0"/>
-      <limit effort="5000.0" velocity="22.0"/>
+      <limit effort="50.0" velocity="22.0"/>
     </joint>
     <joint name="wheel_rr_joint" type="continuous">
@@ -163,20 +226,21 @@
       <child link="wheel_rr"/>
       <axis xyz="0 0 1.0"/>
-      <limit effort="5000.0" velocity="22.0"/>
-    </joint>
-    <material name="black.001">
-      <color rgba="0 0 0 1.0"/>
-    </material>
-    <material name="carpaint_002">
-      <color rgba="0.941177 0.941177 0.941177 1.0"/>
-    </material>
-    <material name="carpaint_002.001">
-      <color rgba="0.941177 0.941177 0.941177 1.0"/>
-    </material>
-    <material name="carpaint_002.002">
-      <color rgba="0.941177 0.941177 0.941177 1.0"/>
-    </material>
-    <material name="carpaint_002.003">
-      <color rgba="0.941177 0.941177 0.941177 1.0"/>
-    </material>
+      <limit effort="50.0" velocity="22.0"/>
+    </joint>
+  <joint name="camera_joint" type="fixed">
+    <axis xyz="0 1 0" />
+    <origin xyz="2.8 0 0.7" rpy="0 0 0"/>
+    <parent link="base_link"/>
+    <child link="camera_link"/>
+  </joint>
+  <joint name="joint_sensor_laser" type="fixed">
+    <origin xyz="1.5 0 1.1" rpy="0 0 0"/>
+    <parent link="base_link"/>
+    <child link="sensor_laser"/>
+  </joint>
+  <joint name="joint_gps" type="fixed">
+    <origin xyz="1.5 0 0.2" rpy="0 0 0"/>
+    <parent link="base_link"/>
+    <child link="gps_link"/>
+  </joint>
   </robot>
